File: HARDWARE/A64-TERES/TERES-PCB3-TOUCH-BTN/Rev.A/TERES-PCB3-TOUCH-BTN_Rev.A.kicad_pcb (KiCad board)
At the start: 2 copper layers, 85 x 12.5 mm, 29 parts, among them P1 CONN_01X05, P2 CONN_01X12

Commit message: Update projects using KiCAD 6.0.7
Other:
- net class Default removed
