File: HARDWARE/A64-TERES/TERES-PCB4-PWR-BTN/Rev.A/PCB4-PWR-BTN_Rev.A.kicad_pcb (KiCad board)
At the start: 2 copper layers, 36 x 10 mm, 8 parts, among them P1 CONN_01X06, SW1 SW_PUSH

Commit message: Update projects using KiCAD 6.0.7
Other:
- net class Default removed
